Commit message: Real Ur5e + hande gripper added

File: dual_ur5e_simulation/src/dual_robot_combined_description/urdf/dual_robots_config.urdf.xacro (robot description, xacro)
@@ -1,4 +1,6 @@
 <?xml version="1.0"?>
 <robot xmlns:xacro="http://www.ros.org/wiki/xacro" name="dual_robots_config">
+    <xacro:arg name="alice_initial_positions_file" default="$(find dual_robot_combined_moveit_config)/config/alice_initial_positions.yaml"/>
+    <xacro:arg name="bob_initial_positions_file" default="$(find dual_robot_combined_moveit_config)/config/bob_initial_positions.yaml"/>
     <!-- Root link -->
     <link name="world"/>
@@ -6,9 +8,9 @@
     <xacro:include filename="robot_with_gripper.urdf.xacro" />
     <!-- alice -->
-    <xacro:ur5e_gripper name="alice_" tf_prefix="alice_" prefix="alice_" parent="world">
+    <xacro:ur5e_gripper name="alice_" tf_prefix="alice_" prefix="alice_" parent="world" initial_positions_file="$(arg alice_initial_positions_file)">
         <origin xyz="0.5 0 0" rpy="0 0 0" />
     </xacro:ur5e_gripper>
     <!-- bob -->
-    <xacro:ur5e_gripper name="bob_" tf_prefix="bob_" prefix="bob_" parent="world">
+    <xacro:ur5e_gripper name="bob_" tf_prefix="bob_" prefix="bob_" parent="world" initial_positions_file="$(arg bob_initial_positions_file)">
         <origin xyz="-0.5 0 0" rpy="0 0 0" />
     </xacro:ur5e_gripper>

File: dual_ur5e_simulation/src/dual_robot_combined_description/urdf/robot_with_gripper.urdf.xacro (robot description, xacro)
@@ -2,5 +2,5 @@
 <robot xmlns:xacro="http://www.ros.org/wiki/xacro">
     <!-- robot name parameter -->
-    <xacro:macro name="ur5e_gripper" params="name tf_prefix prefix parent *origin">
+    <xacro:macro name="ur5e_gripper" params="name tf_prefix prefix parent *origin initial_positions_file">
         <!-- <xacro:arg name="name" default="ur5e" /> -->
         <xacro:arg name="ur_type" default="ur5e" />
@@ -46,6 +46,6 @@
         <xacro:arg name="simulation_controllers" default="" />
         <!-- initial position for simulations (Fake Hardware, Gazebo, Ignition) -->
-        <xacro:arg name="initial_positions_file"
-            default="$(find ur_description)/config/initial_positions.yaml" />
+        <!-- <xacro:arg name="initial_positions_file"
+            default="$(find ur_description)/config/initial_positions.yaml" /> -->
         <!-- convert to property to use substitution in function -->
         <xacro:property name="initial_positions_file" default="$(arg initial_positions_file)" />
